Commit message: Refine URDF with confirmed Hiwonder MechDog specs
Body dimensions updated from RobotShop confirmed specs:
- Standing: 214x126x138mm, weight 560g
- Body platform: 150x85x35mm (estimated from standing height)
- Servos: HPS-0618SG, 8 kg-cm, 180 deg range
- Hip spacing adjusted to match 126mm body width

https://claude.ai/code/session_01NfaFE8A54NEPKJesmAHdmK

File: host/sim/mechdog.urdf (robot description, URDF)
Before this commit: robot mechdog, 14 links, 13 joints
Links:
- link body: mass 0.35 -> 0.40; geometry collision box size=0.150 0.085 0.035; visual box size=0.150 0.085 0.035
- link fl_lower: geometry collision cylinder length=0.060 radius=0.006; visual cylinder length=0.055 radius=0.006
Joints:
- joint fl_hip: origin xyz=0.065 0.040 -0.025 rpy=0 0 0 -> xyz=0.065 0.0425 -0.0175 rpy=0 0 0
- joint ultrasonic_mount: origin xyz=0.095 0 0.010 rpy=0 0 0 -> xyz=0.083 0 0.010 rpy=0 0 0

Commit message: Fix code review issues for physics simulation PR
- P0: SimTransport now inherits from Transport ABC
- P0: Pass physicsClientId to all PyBullet calls (safe for multiple instances)
- P1: Fix URDF FL hip origin asymmetry (was 0.0425/-0.0175, now matches others)
- P1: Fix FL lower leg collision/visual mismatch (both now 0.030/0.060)
- P1: Motion codes 1/2/7/8 now all step physics (hold standing pose)
- P1: speed_factor now multiplies physics steps per CMD cycle
- P1: Add reset_pose() and clear_walls() utility methods
- P1: Tests use reset_pose/clear_walls for proper isolation
- P2: Ultrasonic ray test filters ground plane hits

https://claude.ai/code/session_01NfaFE8A54NEPKJesmAHdmK

File: host/sim/mechdog.urdf (robot description, URDF)
Before this commit: robot mechdog, 14 links, 13 joints
Links:
- link fl_lower: geometry collision cylinder length=0.060 radius=0.006; visual cylinder length=0.060 radius=0.006
Joints:
- joint fl_hip: origin xyz=0.065 0.0425 -0.0175 rpy=0 0 0 -> xyz=0.065 0.040 -0.025 rpy=0 0 0
