Commit message: Update model dimensions to match official MechDog spec (214x126x138mm)
Body platform: 170x60x35mm (was 150x85x35mm)
Hip offset X: 85mm (was 65mm) — matches 214mm overall length
Hip offset Z: 30mm (was 40mm) — matches 126mm overall width
Standing angles: hip=30° knee=-35° (was 17°/34°)

Updated in: kinematics.h, mechdog.urdf, dog3d/state.js, identify_servos.py

Co-Authored-By: Claude Opus 4.6 (1M context) <noreply@anthropic.com>

File: host/sim/mechdog.urdf (robot description, URDF)
Before this commit: robot mechdog, 14 links, 13 joints
Links:
- link body: geometry collision box size=0.170 0.060 0.035; visual box size=0.170 0.060 0.035
Joints:
- joint fl_hip: origin xyz=0.065 0.040 -0.025 rpy=0 0 0 -> xyz=0.085 0.030 -0.025 rpy=0 0 0
- joint fr_hip: origin xyz=0.065 -0.040 -0.025 rpy=0 0 0 -> xyz=0.085 -0.030 -0.025 rpy=0 0 0
- joint rl_hip: origin xyz=-0.065 0.040 -0.025 rpy=0 0 0 -> xyz=-0.085 0.030 -0.025 rpy=0 0 0
- joint rr_hip: origin xyz=-0.065 -0.040 -0.025 rpy=0 0 0 -> xyz=-0.085 -0.030 -0.025 rpy=0 0 0
